File: hardware/kicad/mcu_keys.kicad_sch (KiCad schematic)
At the start: 0 parts

Commit message: sch opt
Other:
- note added: "Keys are active-low; firmware enables internal pull-ups and debounce"
- note added: "Pin 10 PB0 -> KEY1_N -> SW1 -> GND; firmware KEY1_PORT GPIOB KEY1_PIN 0"
- note added: "Pin 11 PB1 -> KEY2_N -> SW2 -> GND; firmware KEY2_PORT GPIOB KEY2_PIN 1"
- note added: "Pin 19 PC1 -> DBG_STRAP/spare; firmware DBG_STRAP_PORT GPIOC DBG_STRAP_PIN 1"
- note added: "Pin 3 PA0/SWIM/BEEP/IR_TIM -> IR_GPIO and SWIM_TP"
- note added: "Pin 4 NRST/PA1 -> NRST_TP; reserve for reset/debug recovery"
- note added: "Pin 9 PD0 -> KEY3_N -> SW3 -> GND; firmware KEY3_PORT GPIOD KEY3_PIN 0"
- note added: "SW1-SW3 use irtool_symbols:SW_Push; TP_SWIM/TP_NRST/TP_VDD/TP_GND use irtool_symbols:TestPoint"
- note added: "U1 STM8L051F3P6 TSSOP-20 active target; use symbol irtool_symbols:STM8L051F3P6"
- note added: "VDD pins -> VDD_MCU; VSS pins -> GND; place C1 100nF close to U1"
- note removed: "Active MCU: STM8L051F3P6; IR/GPIO to gate resistor; KEY1/KEY2/KEY3"
- note removed: "Expose test/debug points: SWIM, NRST, VDD, GND"
- title: MCU and Keys Skeleton -> MCU, Keys and Debug - Electrical Skeleton
Changed lines of the file:
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@@
 (kicad_sch (version 20230121) (generator "codex")
   (paper "A4")
-  (title_block (title "MCU and Keys Skeleton"))
-  (text "Active MCU: STM8L051F3P6; IR/GPIO to gate resistor; KEY1/KEY2/KEY3" (at 35 40 0) (effects (font (size 1.27 1.27))))
-  (text "Expose test/debug points: SWIM, NRST, VDD, GND" (at 35 50 0) (effects (font (size 1.27 1.27))))
+  (title_block (title "MCU, Keys and Debug - Electrical Skeleton"))
+  (hierarchical_label "VDD_MCU" (shape input) (at 25.4 30.48 0)
+    (effects (font (size 1.27 1.27)))
+  )
+  (hierarchical_label "GND" (shape passive) (at 25.4 38.1 0)
+    (effects (font (size 1.27 1.27)))
+  )
+  (hierarchical_label "IR_GPIO" (shape output) (at 25.4 45.72 0)
+    (effects (font (size 1.27 1.27)))
+  )
+  (label "KEY1_N" (at 25.4 66.04 0)
+    (effects (font (size 1.27 1.27)))
+  )
+  (label "KEY2_N" (at 25.4 73.66 0)
+    (effects (font (size 1.27 1.27)))
+  )
+  (label "KEY3_N" (at 25.4 81.28 0)
+    (effects (font (size 1.27 1.27)))
+  )
+  (label "DBG_STRAP" (at 25.4 88.9 0)
+    (effects (font (size 1.27 1.27)))
+  )
+  (label "SWIM_TP" (at 25.4 96.52 0)
+    (effects (font (size 1.27 1.27)))
+  )
+  (label "NRST_TP" (at 25.4 104.14 0)
+    (effects (font (size 1.27 1.27)))
+  )
+  (polyline
+    (pts (xy 58.42 22.86) (xy 172.72 22.86) (xy 172.72 111.76) (xy 58.42 111.76) (xy 58.42 22.86))
+    (stroke (width 0.2) (type default) (color 0 0 0 0))
+  )
+  (text "U1 STM8L051F3P6 TSSOP-20 active target; use symbol irtool_symbols:STM8L051F3P6" (at 63.5 30.48 0)
+    (effects (font (size 1.27 1.27)))
+  )
+  (text "Pin 3 PA0/SWIM/BEEP/IR_TIM -> IR_GPIO and SWIM_TP" (at 63.5 40.64 0)
+    (effects (font (size 1.27 1.27)))
+  )
+  (text "Pin 4 NRST/PA1 -> NRST_TP; reserve for reset/debug recovery" (at 63.5 48.26 0)
+    (effects (font (size 1.27 1.27)))
+  )
+  (text "Pin 10 PB0 -> KEY1_N -> SW1 -> GND; firmware KEY1_PORT GPIOB KEY1_PIN 0" (at 63.5 60.96 0)
+    (effects (font (size 1.27 1.27)))
+  )
+  (text "Pin 11 PB1 -> KEY2_N -> SW2 -> GND; firmware KEY2_PORT GPIOB KEY2_PIN 1" (at 63.5 68.58 0)
+    (effects (font (size 1.27 1.27)))
+  )
+  (text "Pin 9 PD0 -> KEY3_N -> SW3 -> GND; firmware KEY3_PORT GPIOD KEY3_PIN 0" (at 63.5 76.2 0)
+    (effects (font (size 1.27 1.27)))
+  )
+  (text "Pin 19 PC1 -> DBG_STRAP/spare; firmware DBG_STRAP_PORT GPIOC DBG_STRAP_PIN 1" (at 63.5 83.82 0)
+    (effects (font (size 1.27 1.27)))
+  )
+  (text "VDD pins -> VDD_MCU; VSS pins -> GND; place C1 100nF close to U1" (at 63.5 93.98 0)
+    (effects (font (size 1.27 1.27)))
+  )
+  (text "SW1-SW3 use irtool_symbols:SW_Push; TP_SWIM/TP_NRST/TP_VDD/TP_GND use irtool_symbols:TestPoint" (at 63.5 101.6 0)
+    (effects (font (size 1.27 1.27)))
+  )
+  (text "Keys are active-low; firmware enables internal pull-ups and debounce" (at 63.5 109.22 0)
+    (effects (font (size 1.27 1.27)))
+  )
+  (path "/" (page "2"))
 )

Commit message: add pcb
Parts:
- added SW1: KEY1
- added SW2: KEY2
- added SW3: KEY3
- added TP1: SWIM
- added TP2: NRST
- added U1: STM8L051F3P6, Package_SO:TSSOP-20_4.4x6.5mm_P0.65mm
Changed lines of the file:
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@@
     (stroke (width 0.2) (type default) (color 0 0 0 0))
+  )
+  (symbol "irtool_symbols:STM8L051F3P6" (at 111.76 67.31 0) (unit 1) (in_bom yes) (on_board yes)
+    (property "Reference" "U1" (at 111.76 50.8 0) (effects (font (size 1.27 1.27))))
+    (property "Value" "STM8L051F3P6" (at 111.76 86.36 0) (effects (font (size 1.27 1.27))))
+    (property "Footprint" "Package_SO:TSSOP-20_4.4x6.5mm_P0.65mm" (at 111.76 88.9 0) (effects (font (size 1.27 1.27)) hide))
+    (pin "1")
+    (pin "3")
+    (pin "4")
+    (pin "8")
+    (pin "9")
+    (pin "10")
+    (pin "11")
+    (pin "19")
+    (pin "20")
+    (instances
+      (project "remote"
+        (path "/4a7a9960-a803-42d7-9baf-7a81f45e2001"
+          (reference "U1")
+          (unit 1)
+        )
+      )
+    )
+  )
+  (symbol "irtool_symbols:SW_Push" (at 154.94 60.96 0) (unit 1) (in_bom yes) (on_board yes)
+    (property "Reference" "SW1" (at 154.94 57.15 0) (effects (font (size 1.27 1.27))))
+    (property "Value" "KEY1" (at 154.94 64.77 0) (effects (font (size 1.27 1.27))))
+    (pin "1")
+    (pin "2")
+    (instances (project "remote" (path "/4a7a9960-a803-42d7-9baf-7a81f45e2001" (reference "SW1") (unit 1))))
+  )
+  (symbol "irtool_symbols:SW_Push" (at 154.94 71.12 0) (unit 1) (in_bom yes) (on_board yes)
+    (property "Reference" "SW2" (at 154.94 67.31 0) (effects (font (size 1.27 1.27))))
+    (property "Value" "KEY2" (at 154.94 74.93 0) (effects (font (size 1.27 1.27))))
+    (pin "1")
+    (pin "2")
+    (instances (project "remote" (path "/4a7a9960-a803-42d7-9baf-7a81f45e2001" (reference "SW2") (unit 1))))
+  )
+  (symbol "irtool_symbols:SW_Push" (at 154.94 81.28 0) (unit 1) (in_bom yes) (on_board yes)
+    (property "Reference" "SW3" (at 154.94 77.47 0) (effects (font (size 1.27 1.27))))
+    (property "Value" "KEY3" (at 154.94 85.09 0) (effects (font (size 1.27 1.27))))
+    (pin "1")
+    (pin "2")
+    (instances (project "remote" (path "/4a7a9960-a803-42d7-9baf-7a81f45e2001" (reference "SW3") (unit 1))))
+  )
+  (symbol "irtool_symbols:TestPoint" (at 68.58 45.72 0) (unit 1) (in_bom no) (on_board yes)
+    (property "Reference" "TP1" (at 68.58 43.18 0) (effects (font (size 1.27 1.27))))
+    (property "Value" "SWIM" (at 68.58 48.26 0) (effects (font (size 1.27 1.27))))
+    (pin "1")
+    (instances (project "remote" (path "/4a7a9960-a803-42d7-9baf-7a81f45e2001" (reference "TP1") (unit 1))))
+  )
+  (symbol "irtool_symbols:TestPoint" (at 68.58 55.88 0) (unit 1) (in_bom no) (on_board yes)
+    (property "Reference" "TP2" (at 68.58 53.34 0) (effects (font (size 1.27 1.27))))
+    (property "Value" "NRST" (at 68.58 58.42 0) (effects (font (size 1.27 1.27))))
+    (pin "1")
+    (instances (project "remote" (path "/4a7a9960-a803-42d7-9baf-7a81f45e2001" (reference "TP2") (unit 1))))
   )
   (text "U1 STM8L051F3P6 TSSOP-20 active target; use symbol irtool_symbols:STM8L051F3P6" (at 63.5 30.48 0)

Commit message: pcb opt
Parts:
- added C4: 100nF
- added RD10, RD11, RD5, RD6, RD7, RD8, RD9: 100K
- added SW1: KEY1
- added SW2: KEY2
- added SW3: KEY3
- added TP1: SWIM
- added TP3: VDD
- added TP4: GND
- added TP5: DBG
- RD1: renamed from SW1; value KEY1 -> 100K
- RD2: renamed from SW2; value KEY2 -> 100K
- RD3: renamed from SW3; value KEY3 -> 100K
- RD4: renamed from TP1; value SWIM -> 100K; now in the parts list
Other:
- note added: "Active-low keys to GND; internal pull-ups and debounce handled in firmware"
- note added: "All 20 MCU pins connected. Unused pins (PC7/PA2/PA3/PB7/PB2-PB6/PC4/PC5) tied to GND via 100K pull-down resistors for low power."
- note added: "Pin map: PA0=IR_GPIO/SWIM, PB0=KEY1_N, PB1=KEY2_N, PD0=KEY3_N, PC1=DBG_STRAP"
- note removed: "Keys are active-low; firmware enables internal pull-ups and debounce"
- note removed: "Pin 10 PB0 -> KEY1_N -> SW1 -> GND; firmware KEY1_PORT GPIOB KEY1_PIN 0"
- note removed: "Pin 11 PB1 -> KEY2_N -> SW2 -> GND; firmware KEY2_PORT GPIOB KEY2_PIN 1"
- note removed: "Pin 19 PC1 -> DBG_STRAP/spare; firmware DBG_STRAP_PORT GPIOC DBG_STRAP_PIN 1"
- note removed: "Pin 3 PA0/SWIM/BEEP/IR_TIM -> IR_GPIO and SWIM_TP"
- note removed: "Pin 4 NRST/PA1 -> NRST_TP; reserve for reset/debug recovery"
- note removed: "Pin 9 PD0 -> KEY3_N -> SW3 -> GND; firmware KEY3_PORT GPIOD KEY3_PIN 0"
- note removed: "SW1-SW3 use irtool_symbols:SW_Push; TP_SWIM/TP_NRST/TP_VDD/TP_GND use irtool_symbols:TestPoint"
- note removed: "U1 STM8L051F3P6 TSSOP-20 active target; use symbol irtool_symbols:STM8L051F3P6"
- note removed: "VDD pins -> VDD_MCU; VSS pins -> GND; place C1 100nF close to U1"
- title: MCU, Keys and Debug - Electrical Skeleton -> MCU, Keys and Debug
