File: hardware/kicad/remote.kicad_pcb (KiCad board)
At the start: 2 copper layers, 110 x 80 mm, 18 parts, among them Q1 IRLML2502, SW1 KEY1, SW2 KEY2, SW3 KEY3, U1 STM8L051F3P6

Commit message: pcb opt
Routing:
- net IR_GATE: track 0.00 -> 26.0 mm
- net IR_LED_A: track 0.00 -> 25.9 mm
- net GND: track 0.00 -> 23.9 mm
- net IR_LED_K: track 0.00 -> 19.2 mm
- net VDD_MCU: track 0.00 -> 18.5 mm
- net IR_GPIO: track 0.00 -> 8.95 mm
Other:
- board text added: "CR2032 BACK SIDE HOLDER"
- board text added: "DEBUG / PROGRAMMING PADS"
- board text added: "KEY ZONE"
- board text added: "MCU + IR DRIVER ZONE"
Changed lines of the file:
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@@
     (pad "1" smd circle (at 0 0) (size 1.8 1.8) (layers "F.Cu" "F.Mask") (net 12 "DBG_STRAP"))
+  )
+  (segment (start 127.2 74) (end 136.15 74) (width 0.25) (layer "F.Cu") (net 3))
+  (segment (start 127.65 74) (end 142.8 74) (width 0.25) (layer "F.Cu") (net 4))
+  (segment (start 132.85 60) (end 158.73 60) (width 0.4) (layer "F.Cu") (net 8))
+  (segment (start 161.27 60) (end 147.2 73.05) (width 0.4) (layer "F.Cu") (net 9))
+  (segment (start 138.15 81) (end 147.2 74.95) (width 0.25) (layer "F.Cu") (net 4))
+  (segment (start 139.85 81) (end 143 81) (width 0.25) (layer "F.Cu") (net 1))
+  (segment (start 96.15 62) (end 110.2 74.075) (width 0.3) (layer "F.Cu") (net 2))
+  (segment (start 97.85 62) (end 110.2 78.625) (width 0.3) (layer "F.Cu") (net 1))
+  (gr_rect (start 90 52) (end 166 86) (stroke (width 0.08) (type dash)) (fill none) (layer "Dwgs.User"))
+  (gr_rect (start 92 95) (end 138 111) (stroke (width 0.08) (type dash)) (fill none) (layer "Dwgs.User"))
+  (gr_rect (start 72 40) (end 134 50) (stroke (width 0.08) (type dash)) (fill none) (layer "Dwgs.User"))
+  (gr_text "MCU + IR DRIVER ZONE" (at 128 54 0) (layer "Dwgs.User")
+    (effects (font (size 1.2 1.2) (thickness 0.15)))
+  )
+  (gr_text "KEY ZONE" (at 115 97 0) (layer "Dwgs.User")
+    (effects (font (size 1.2 1.2) (thickness 0.15)))
+  )
+  (gr_text "DEBUG / PROGRAMMING PADS" (at 103 42 0) (layer "Dwgs.User")
+    (effects (font (size 1.2 1.2) (thickness 0.15)))
+  )
+  (gr_text "CR2032 BACK SIDE HOLDER" (at 82 99 0) (layer "Dwgs.User")
+    (effects (font (size 1.2 1.2) (thickness 0.15)))
   )
   (gr_line (start 60 35) (end 170 35) (stroke (width 0.1) (type default)) (layer "Edge.Cuts"))

Commit message: pcb opt
Parts:
- removed the C2 at (97.0, 68.0)
- removed the C3 at (97.0, 74.0)
- removed R3: R_PD 1M, irtool:R0603_PLACEHOLDER
- added H1: M2, MountingHole:MountingHole_2.2mm_M2, F.Cu at (15.0, 50.0)
- added H2: M2, MountingHole:MountingHole_2.2mm_M2, F.Cu at (175.0, 50.0)
- added H3: M2, MountingHole:MountingHole_2.2mm_M2, F.Cu at (15.0, 115.0)
- added H4: M2, MountingHole:MountingHole_2.2mm_M2, F.Cu at (175.0, 115.0)
- added TP1: SWIM, irtool:TP1_SWIM, F.Cu at (85.0, 55.0)
- added TP2: NRST, irtool:TP2_NRST, F.Cu at (92.0, 55.0)
- added TP3: VDD, irtool:TP3_VDD, F.Cu at (99.0, 55.0)
- BT1: renamed from SW3; value KEY3 -> CR2032; footprint irtool:SW_PLACEHOLDER -> irtool:BT1_CR2032_Holder; moved to B.Cu
- C1: renamed from BT1; value CR2032 Holder -> 100nF; footprint irtool:BT1_CR2032_PLACEHOLDER -> irtool:C1_100nF_0402; moved to F.Cu
- C2: renamed from SW1; value KEY1 -> 4.7uF; footprint irtool:SW_PLACEHOLDER -> irtool:C2_4u7F_0603
- C3: renamed from SW2; value KEY2 -> 47uF OPT; footprint irtool:SW_PLACEHOLDER -> irtool:C3_47uF_OPT
- D1: value IR_LED -> 940nm; footprint irtool:LED_D5_PLACEHOLDER -> irtool:D1_IR_LED_5mm
- Q1: footprint irtool:Q1_SOT23_PLACEHOLDER -> irtool:Q1_IRLML2502_SOT23
- R1: renamed from C1; value 100n -> 10-22R; footprint irtool:C0603_PLACEHOLDER -> irtool:R1_IR_LED_0603
- R2: renamed from R1; value R_LED -> 100R; footprint irtool:R0603_PLACEHOLDER -> irtool:R2_GATE_100R_0603
- R_PD: renamed from R2; value R_GATE -> 1M; footprint irtool:R0603_PLACEHOLDER -> irtool:R_PD_1M_0603
- SW1: renamed from TP1; value SWIM -> KEY1; footprint irtool:TP_PLACEHOLDER -> irtool:SW1_KEY1
- SW2: renamed from TP2; value NRST -> KEY2; footprint irtool:TP_PLACEHOLDER -> irtool:SW2_KEY2
- SW3: renamed from TP3; value VDD -> KEY3; footprint irtool:TP_PLACEHOLDER -> irtool:SW3_KEY3
- TP4: footprint irtool:TP_PLACEHOLDER -> irtool:TP4_GND
- TP5: footprint irtool:TP_PLACEHOLDER -> irtool:TP5_DBG
- U1: footprint irtool:U1_STM8L051F3P6_TSSOP20_PLACEHOLDER -> irtool:U1_STM8L051F3P6_TSSOP20
- moved SW3 64.0 mm to (115.0, 110.0)
- moved SW2 61.3 mm to (135.0, 100.0)
- moved BT1 60.8 mm to (75.0, 75.0)
- moved R1 59.0 mm to (155.0, 73.0)
- moved SW1 56.6 mm to (115.0, 100.0)
- moved C3 20.6 mm to (99.0, 90.0)
- moved TP5 19.2 mm to (113.0, 55.0)
- moved TP4 18.4 mm to (106.0, 55.0)
- moved C2 17.1 mm to (99.0, 86.0)
- moved C1 17.0 mm to (99.0, 82.0), turned to 0 degrees
- moved D1 15.5 mm to (164.0, 75.0)
- moved R_PD 14.0 mm to (132.0, 60.0)
- moved Q1 12.8 mm to (135.0, 66.0)
- moved U1 10.2 mm to (105.0, 75.0)
- moved R2 8.06 mm to (128.0, 67.0)
Connections:
- BT1 pad 1: KEY3_N -> VDD_MCU
- C2 pad 1: KEY1_N -> VDD_MCU
- C3 pad 1: KEY2_N -> VDD_MCU
- R1 pad 2: GND -> IR_LED_A
- R2 pad 1: VDD_MCU -> IR_GPIO
- R2 pad 2: IR_LED_A -> IR_GATE
- R_PD pad 1: IR_GPIO -> IR_GATE
- R_PD pad 2: IR_GATE -> GND
- SW1 pad 1: SWIM_TP -> KEY1_N
- SW2 pad 1: NRST_TP -> KEY2_N
- SW3 pad 1: VDD_MCU -> KEY3_N
Routing:
- net VDD_MCU: track 18.5 -> 122.2 mm
- net IR_GPIO: track 8.95 -> 53.0 mm
- net KEY3_N: track 0.00 -> 43.8 mm
- net KEY2_N: track 0.00 -> 42.4 mm
- net NRST_TP: track 0.00 -> 27.0 mm
- net DBG_STRAP: track 0.00 -> 23.9 mm
- net GND: track 23.9 -> 0.00 mm
- net KEY1_N: track 0.00 -> 22.1 mm
- net IR_LED_A: track 25.9 -> 4.05 mm
- net IR_GATE: track 26.0 -> 13.8 mm
- net IR_LED_K: track 19.2 -> 31.0 mm
- added copper zone on B.Cu, net GND
- added copper zone on F.Cu, net GND
Other:
- net class Default added: clearance 0.2, trace_width 0.25, via_dia 0.6, via_drill 0.3
- net class Power added: clearance 0.25, trace_width 0.5, via_dia 0.8, via_drill 0.4
- board text added: "+"
- board text added: "-"
- board text added: "CR2032"
- board text added: "IR ->"
- board text added: "KEY1"
- board text added: "KEY2"
- board text added: "KEY3"
- board text added: "STM8L051F3P6 IR Remote"
- board text added: "TP1 SWIM"
- board text added: "TP2 NRST"
- board text added: "TP3 VDD"
- board text added: "TP4 GND"
- board text added: "TP5 DBG"
- board text removed: "CR2032 BACK SIDE HOLDER"
- board text removed: "DEBUG / PROGRAMMING PADS"
- board text removed: "KEY ZONE"
- board text removed: "MCU + IR DRIVER ZONE"
- board text removed: "PCB skeleton only No final placement/routing claims"
