File: hardware/kicad/remote.kicad_sch (KiCad schematic)
At the start: 0 parts

Commit message: pcb opt
Other:
- note added: "All 20 MCU pins connected on sheet 2. Unused pins terminated via 100K to GND."
- note added: "Hierarchy: left = MCU+Keys+Debug, right = CR2032 power and IRLML2502 driver"
- note added: "PWR_FLAG symbols satisfy ERC: VDD_MCU driven by BT1 CR2032, GND is battery return."
- note added: "Pin map: PA0=IR_GPIO/SWIM, PB0=KEY1_N, PB1=KEY2_N, PD0=KEY3_N, PC1=DBG_STRAP"
- note removed: "Code/schematic pin map: PA0=IR_GPIO/SWIM, PB0=KEY1_N, PB1=KEY2_N, PD0=KEY3_N, PC1=DBG_STRAP"
- note removed: "Hierarchy: left sheet = MCU+Keys+Debug, right sheet = CR2032 power and IRLML2502 driver"
- note removed: "Inter-sheet nets refined in this pass: VDD_MCU, GND, IR_GPIO"
- note removed: "Project-local symbol library: irtool_symbols (see sym-lib-table)"
- note removed: "Review scope only: no PCB, no production library pack, no bench-verified current/range claims"
Changed lines of the file:
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@@
     (comment 1 "Root schematic for remote.kicad_pro")
     (comment 2 "Active target: STM8L051F3P6 + IRLML2502 + CR2032")
-    (comment 3 "First-pass review schematic; no PCB/layout claims")
+    (comment 3 "Hierarchy: mcu_keys (page 2), power_ir (page 3)")
   )
+  ;; ---- Child sheet 1: MCU + Keys + Debug ----
   (sheet
     (at 35.56 45.72 0)
@@
     (stroke (width 0.1524) (type solid) (color 0 0 0 0))
     (fill (color 0 0 0 0.0000))
-    (property "Sheetname" "MCU_Keys_Debug" (at 38.1 46.99 0)
-      (effects (font (size 1.27 1.27)) (justify left bottom))
-    )
-    (property "Sheetfile" "mcu_keys.kicad_sch" (at 38.1 118.11 0)
-      (effects (font (size 1.27 1.27)) (justify left top))
-    )
-    (pin "VDD_MCU" input (at 116.84 60.96 0)
-      (effects (font (size 1.27 1.27)) (justify right))
-    )
-    (pin "GND" passive (at 116.84 71.12 0)
-      (effects (font (size 1.27 1.27)) (justify right))
-    )
-    (pin "IR_GPIO" output (at 116.84 81.28 0)
-      (effects (font (size 1.27 1.27)) (justify right))
-    )
-    (instances
-      (project "remote"
-        (path "/2e068f12-6b3d-45d8-a7a2-3d3e7c6f1001/2e068f12-6b3d-45d8-a7a2-3d3e7c6f1002"
-          (page "2")
-        )
-      )
-    )
+    (property "Sheetname" "MCU_Keys_Debug" (at 38.1 46.99 0) (effects (font (size 1.27 1.27)) (justify left bottom)))
+    (property "Sheetfile" "mcu_keys.kicad_sch" (at 38.1 118.11 0) (effects (font (size 1.27 1.27)) (justify left top)))
+    (pin "VDD_MCU" input (at 116.84 60.96 0) (effects (font (size 1.27 1.27)) (justify right)))
+    (pin "GND" passive (at 116.84 71.12 0) (effects (font (size 1.27 1.27)) (justify right)))
+    (pin "IR_GPIO" output (at 116.84 81.28 0) (effects (font (size 1.27 1.27)) (justify right)))
+    (instances (project "remote" (path "/2e068f12-6b3d-45d8-a7a2-3d3e7c6f1001/2e068f12-6b3d-45d8-a7a2-3d3e7c6f1002" (page "2"))))
   )
+  ;; ---- Child sheet 2: Power + IR Driver ----
   (sheet
     (at 149.86 45.72 0)
@@
     (stroke (width 0.1524) (type solid) (color 0 0 0 0))
     (fill (color 0 0 0 0.0000))
-    (property "Sheetname" "Power_IR_Driver" (at 152.4 46.99 0)
-      (effects (font (size 1.27 1.27)) (justify left bottom))
-    )
-    (property "Sheetfile" "power_ir.kicad_sch" (at 152.4 118.11 0)
-      (effects (font (size 1.27 1.27)) (justify left top))
-    )
-    (pin "VDD_MCU" input (at 149.86 60.96 180)
-      (effects (font (size 1.27 1.27)) (justify left))
-    )
-    (pin "GND" passive (at 149.86 71.12 180)
-      (effects (font (size 1.27 1.27)) (justify left))
-    )
-    (pin "IR_GPIO" input (at 149.86 81.28 180)
-      (effects (font (size 1.27 1.27)) (justify left))
-    )
-    (instances
-      (project "remote"
-        (path "/2e068f12-6b3d-45d8-a7a2-3d3e7c6f1001/2e068f12-6b3d-45d8-a7a2-3d3e7c6f1003"
-          (page "3")
-        )
-      )
-    )
+    (property "Sheetname" "Power_IR_Driver" (at 152.4 46.99 0) (effects (font (size 1.27 1.27)) (justify left bottom)))
+    (property "Sheetfile" "power_ir.kicad_sch" (at 152.4 118.11 0) (effects (font (size 1.27 1.27)) (justify left top)))
+    (pin "VDD_MCU" input (at 149.86 60.96 180) (effects (font (size 1.27 1.27)) (justify left)))
+    (pin "GND" passive (at 149.86 71.12 180) (effects (font (size 1.27 1.27)) (justify left)))
+    (pin "IR_GPIO" input (at 149.86 81.28 180) (effects (font (size 1.27 1.27)) (justify left)))
+    (instances (project "remote" (path "/2e068f12-6b3d-45d8-a7a2-3d3e7c6f1001/2e068f12-6b3d-45d8-a7a2-3d3e7c6f1003" (page "3"))))
   )
-  (wire
-    (pts (xy 116.84 60.96) (xy 149.86 60.96))
-    (stroke (width 0) (type default) (color 0 0 0 0))
+  ;; ---- Inter-sheet wires ----
+  (wire (pts (xy 116.84 60.96) (xy 149.86 60.96)) (stroke (width 0) (type default) (color 0 0 0 0)))
+  (wire (pts (xy 116.84 71.12) (xy 149.86 71.12)) (stroke (width 0) (type default) (color 0 0 0 0)))
+  (wire (pts (xy 116.84 81.28) (xy 149.86 81.28)) (stroke (width 0) (type default) (color 0 0 0 0)))
+  ;; ---- PWR_FLAG instances for ERC ----
+  (symbol "irtool_symbols:PWR_FLAG" (at 133.35 58.42 0) (unit 1) (in_bom yes) (on_board yes)
+    (property "Reference" "#FLG1" (at 133.35 56.515 0) (effects (font (size 1.27 1.27)) hide))
+    (property "Value" "PWR_FLAG" (at 133.35 60.325 0) (effects (font (size 1.27 1.27)) hide))
+    (pin "1")
+    (instances (project "remote" (path "/2e068f12-6b3d-45d8-a7a2-3d3e7c6f1001" (reference "#FLG1") (unit 1))))
   )
-  (wire
-    (pts (xy 116.84 71.12) (xy 149.86 71.12))
-    (stroke (width 0) (type default) (color 0 0 0 0))
+  (symbol "irtool_symbols:PWR_FLAG" (at 133.35 68.58 0) (unit 1) (in_bom yes) (on_board yes)
+    (property "Reference" "#FLG2" (at 133.35 66.675 0) (effects (font (size 1.27 1.27)) hide))
+    (property "Value" "PWR_FLAG" (at 133.35 70.485 0) (effects (font (size 1.27 1.27)) hide))
+    (pin "1")
+    (instances (project "remote" (path "/2e068f12-6b3d-45d8-a7a2-3d3e7c6f1001" (reference "#FLG2") (unit 1))))
   )
-  (wire
-    (pts (xy 116.84 81.28) (xy 149.86 81.28))
-    (stroke (width 0) (type default) (color 0 0 0 0))
-  )
-  (text "Project-local symbol library: irtool_symbols (see sym-lib-table)" (at 36.83 25.4 0)
-    (effects (font (size 1.27 1.27)))
-  )
-  (text "Code/schematic pin map: PA0=IR_GPIO/SWIM, PB0=KEY1_N, PB1=KEY2_N, PD0=KEY3_N, PC1=DBG_STRAP" (at 36.83 31.75 0)
-    (effects (font (size 1.27 1.27)))
-  )
-  (text "Hierarchy: left sheet = MCU+Keys+Debug, right sheet = CR2032 power and IRLML2502 driver" (at 36.83 38.1 0)
-    (effects (font (size 1.27 1.27)))
-  )
-  (text "Inter-sheet nets refined in this pass: VDD_MCU, GND, IR_GPIO" (at 36.83 127 0)
-    (effects (font (size 1.27 1.27)))
-  )
-  (text "Review scope only: no PCB, no production library pack, no bench-verified current/range claims" (at 36.83 133.35 0)
-    (effects (font (size 1.27 1.27)))
-  )
+  (wire (pts (xy 133.35 58.42) (xy 133.35 60.96)) (stroke (width 0) (type default) (color 0 0 0 0)))
+  (wire (pts (xy 133.35 68.58) (xy 133.35 71.12)) (stroke (width 0) (type default) (color 0 0 0 0)))
+  ;; ---- Annotations ----
+  (text "PWR_FLAG symbols satisfy ERC: VDD_MCU driven by BT1 CR2032, GND is battery return." (at 36.83 25.4 0) (effects (font (size 1.27 1.27))))
+  (text "Pin map: PA0=IR_GPIO/SWIM, PB0=KEY1_N, PB1=KEY2_N, PD0=KEY3_N, PC1=DBG_STRAP" (at 36.83 31.75 0) (effects (font (size 1.27 1.27))))
+  (text "Hierarchy: left = MCU+Keys+Debug, right = CR2032 power and IRLML2502 driver" (at 36.83 38.1 0) (effects (font (size 1.27 1.27))))
+  (text "All 20 MCU pins connected on sheet 2. Unused pins terminated via 100K to GND." (at 36.83 127 0) (effects (font (size 1.27 1.27))))
   (path "/" (page "1"))
 )
